File: Eagle/SRAM 4MB 2048kbx8 CPLD proto.brd (EAGLE design)
At the start: 100.1 x 58 mm, 28 parts, among them IC13 BS62LV1600EIP55-10ZSXI, IC14 BS62LV1600EIP55-10ZSXI, IC2 74LS245DW, IC3 74LS245DW, IC4 74LS245DW, IC5 XC9536_44PLCC, U1 M48Z02-70PC1, U2 LD6815TD/33H, X1 PCMCIA female

Commit message: New version of board
Parts:
- renumbered IC13 to IC6, IC14 to IC7, U1 to IC1, U2 to IC8
Other:
- outline, holes or cut-outs redrawn
