File: board/v1.2/Eagle/SRAM 4MB 2048kbx8 CPLD_v1_2.brd (EAGLE design)
At the start: 65.8 x 49.7 mm, 23 parts, among them IC1 LD6815TD/33H, IC2 74LS245MTC, IC3 74LS245MTC, IC4 74LS245MTC, IC5 XC9536_44VQ, IC6 BS62LV1600EIP55-10ZSXI, IC7 BS62LV1600EIP55-10ZSXI, SW1 RAM/Disk, X1 PCMCIA female

Commit message: New version of board v2.1
Parts:
- moved X1 1.35 mm to (99.9, 42.0)
Routing:
- net +5V: track 176.8 -> 171.9 mm
- net D7: track 77.9 -> 75.9 mm
- net A5: track 105.7 -> 103.8 mm
- net D4: track 66.3 -> 64.5 mm
- net A18: track 57.9 -> 56.3 mm
- net A0: track 62.8 -> 61.1 mm
- net D1: track 79.3 -> 77.8 mm
- net D2: track 82.5 -> 81.0 mm
- net A4: track 99.1 -> 97.6 mm
- net A3: track 99.2 -> 97.7 mm
- net CE1#: track 74.5 -> 73.1 mm
- net D6: track 78.3 -> 76.9 mm
- net A1: track 100.1 -> 98.7 mm
- net REG#: track 62.6 -> 61.2 mm
- net A2: track 99.7 -> 98.3 mm
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Other:
- board size 65.8 x 49.7 mm -> 64.4 x 49.7 mm
